File: src/ModbusRTU-Test-Shield.kicad_sch (KiCad schematic)
At the start: 40 parts, among them J1 Conn_01x08_UNO_Digital_1, J2 Conn_01x10_UNO_Digital_2, J3 Conn_01x08_UNO_Power, J4 Conn_01x06_UNO_Analog, J5 Screw_Terminal_01x03, J6 6P6C, SW1 RESET, SW2 BUTTON1, SW3 BUTTON2, SW4 SW_DPDT_x2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

Commit message: Updated the schematic and board to use the new footprints and models.
Parts:
- D11: footprint Diode_THT:D_DO-41_SOD81_P10.16mm_Horizontal -> Project_Footprints:D_DO-41_SOD81_P10.16mm_Horizontal
- SW4: footprint Button_Switch_THT:SW_E-Switch_EG1271_SPDT -> Project_Footprints:SW_CK_OS202011MS2Qx1_DPDT; Manufacturer (none) -> C&K; Part Number (none) -> OS202011MS2QN1
Changed lines of the file:
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@@
       (effects (font (size 1.27 1.27)))
     )
-    (property "Footprint" "Button_Switch_THT:SW_E-Switch_EG1271_SPDT" (at 254 190.5 0)
+    (property "Footprint" "Project_Footprints:SW_CK_OS202011MS2Qx1_DPDT" (at 254 190.5 0)
       (effects (font (size 1.27 1.27)) hide)
     )
-    (property "Datasheet" "~" (at 254 190.5 0)
+    (property "Datasheet" "https://www.ckswitches.com/media/1428/os.pdf" (at 254 190.5 0)
+      (effects (font (size 1.27 1.27)) hide)
+    )
+    (property "Manufacturer" "C&K" (at 254 190.5 0)
+      (effects (font (size 1.27 1.27)) hide)
+    )
+    (property "Part Number" "OS202011MS2QN1" (at 254 190.5 0)
+      (effects (font (size 1.27 1.27)) hide)
+    )
+    (property "Description" "DPDT Slide Switch" (at 254 190.5 0)
+      (effects (font (size 1.27 1.27)) hide)
+    )
+    (property "Item" "" (at 254 190.5 0)
       (effects (font (size 1.27 1.27)) hide)
     )
@@
       (effects (font (size 1.27 1.27)))
     )
-    (property "Footprint" "Button_Switch_THT:SW_E-Switch_EG1271_SPDT" (at 254 154.94 0)
+    (property "Footprint" "Project_Footprints:SW_CK_OS202011MS2Qx1_DPDT" (at 254 154.94 0)
       (effects (font (size 1.27 1.27)) hide)
     )
-    (property "Datasheet" "~" (at 254 154.94 0)
+    (property "Datasheet" "https://www.ckswitches.com/media/1428/os.pdf" (at 254 154.94 0)
+      (effects (font (size 1.27 1.27)) hide)
+    )
+    (property "Manufacturer" "C&K" (at 254 154.94 0)
+      (effects (font (size 1.27 1.27)) hide)
+    )
+    (property "Part Number" "OS202011MS2QN1" (at 254 154.94 0)
+      (effects (font (size 1.27 1.27)) hide)
+    )
+    (property "Description" "DPDT Slide Switch" (at 254 154.94 0)
+      (effects (font (size 1.27 1.27)) hide)
+    )
+    (property "Item" "" (at 254 154.94 0)
       (effects (font (size 1.27 1.27)) hide)
     )
@@
       (effects (font (size 1.27 1.27)))
     )
-    (property "Footprint" "Diode_THT:D_DO-41_SOD81_P10.16mm_Horizontal" (at 72.39 226.06 0)
+    (property "Footprint" "Project_Footprints:D_DO-41_SOD81_P10.16mm_Horizontal" (at 72.39 226.06 0)
       (effects (font (size 1.27 1.27)) hide)
     )
@@
       (effects (font (size 1.27 1.27)) hide)
     )
+    (property "Manufacturer" "" (at 72.39 226.06 0)
+      (effects (font (size 1.27 1.27)) hide)
+    )
+    (property "Part Number" "" (at 72.39 226.06 0)
+      (effects (font (size 1.27 1.27)) hide)
+    )
+    (property "Description" "" (at 72.39 226.06 0)
+      (effects (font (size 1.27 1.27)) hide)
+    )
+    (property "Item" "" (at 72.39 226.06 0)
+      (effects (font (size 1.27 1.27)) hide)
+    )

Commit message: Completed third draft.
Parts:
- C1: now not fitted; now left out of the parts list
- C2, C3, C4, C5, C6: footprint Capacitor_THT:CP_Radial_D5.0mm_P2.50mm -> Project_Footprints:CP_Radial_D5.0mm_P2.50mm
- D1: footprint LED_THT:LED_D3.0mm -> Project_Footprints:LED_D3.0mm; Label (none) -> LED4
- D10: footprint LED_THT:LED_D3.0mm -> Project_Footprints:LED_D3.0mm; Label (none) -> RX
- D2: footprint LED_THT:LED_D3.0mm -> Project_Footprints:LED_D3.0mm; Label (none) -> LED3
- D3: footprint LED_THT:LED_D3.0mm -> Project_Footprints:LED_D3.0mm; Label (none) -> LED2
- D4: footprint LED_THT:LED_D3.0mm -> Project_Footprints:LED_D3.0mm; Label (none) -> LED1
- D5: footprint LED_THT:LED_D3.0mm -> Project_Footprints:LED_D3.0mm; Label (none) -> DE
- D6, D7: footprint Diode_THT:D_DO-35_SOD27_P7.62mm_Horizontal -> Project_Footprints:D_DO-35_SOD27_P7.62mm_Horizontal
- D8: footprint LED_THT:LED_D3.0mm -> Project_Footprints:LED_D3.0mm; Label (none) -> PWR
- D9: footprint LED_THT:LED_D3.0mm -> Project_Footprints:LED_D3.0mm; Label (none) -> TX
- R1, R2, R3, R4, R5, R6, R7, R8, R9: footprint Resistor_THT:R_Axial_DIN0204_L3.6mm_D1.6mm_P7.62mm_Horizontal -> Project_Footprints:R_Axial_DIN0204_L3.6mm_D1.6mm_P7.62mm_Horizontal
- RV1: Label POT 1 -> POT1
- RV2: Label POT 2 -> POT2
- SW2: Label BUTTON 1 -> BTN1
- SW3: Label BUTTON 2 -> BTN2
- U1: value LT1785AxN8 -> LT1785; footprint Package_DIP:DIP-8_W7.62mm_Socket -> Project_Footprints:DIP-8_W7.62mm_Socket
- U2: footprint Package_DIP:DIP-16_W7.62mm_Socket -> Project_Footprints:DIP-16_W7.62mm_Socket

Commit message: Completed fourth draft.
Parts:
- removed C1: 0.1uF, Capacitor_THT:C_Disc_D3.8mm_W2.6mm_P2.50mm, symbol Device:C
- added C1: 1uF, Project_Footprints:CP_Radial_D4.0mm_P1.50mm, symbol Device:C_Polarized_Small
- C2: renamed from C6; footprint Project_Footprints:CP_Radial_D5.0mm_P2.50mm -> Project_Footprints:CP_Radial_D4.0mm_P1.50mm; Manufacturer (none) -> KEMET; Part Number (none) -> ESS105M050AB2EA
- C3: renamed from C4; footprint Project_Footprints:CP_Radial_D5.0mm_P2.50mm -> Project_Footprints:CP_Radial_D4.0mm_P1.50mm; Manufacturer (none) -> KEMET; Part Number (none) -> ESS105M050AB2EA
- C4: renamed from C3; footprint Project_Footprints:CP_Radial_D5.0mm_P2.50mm -> Project_Footprints:CP_Radial_D4.0mm_P1.50mm; Manufacturer (none) -> KEMET; Part Number (none) -> ESS105M050AB2EA
- C5: footprint Project_Footprints:CP_Radial_D5.0mm_P2.50mm -> Project_Footprints:CP_Radial_D4.0mm_P1.50mm; Manufacturer (none) -> KEMET; Part Number (none) -> ESS105M050AB2EA
- C6: renamed from C2; footprint Project_Footprints:CP_Radial_D5.0mm_P2.50mm -> Project_Footprints:CP_Radial_D4.0mm_P1.50mm; Manufacturer (none) -> KEMET; Part Number (none) -> ESS105M050AB2EA
- D1: Label LED4 -> L1; Manufacturer (none) -> Würth Elektronik; Part Number (none) -> 151031YS06000
- D10: renamed from D7; value D_Schottky -> BAT43; Manufacturer (none) -> Vishay; Part Number (none) -> BAT43-TAP
- D11: value D_Schottky -> SB260S; Manufacturer (none) -> Vishay; Part Number (none) -> SB260S-E3/54
- D2: Label LED3 -> L2; Manufacturer (none) -> Würth Elektronik; Part Number (none) -> 151031YS06000
- D3: Label LED2 -> L3; Manufacturer (none) -> Würth Elektronik; Part Number (none) -> 151031YS06000
- D4: Label LED1 -> L4; Manufacturer (none) -> Würth Elektronik; Part Number (none) -> 151031YS06000
- D5: renamed from D8; Label PWR -> ON; Manufacturer (none) -> Würth Elektronik; Part Number (none) -> 151031VS04000
- D6: renamed from D5; Manufacturer (none) -> Würth Elektronik; Part Number (none) -> 151031YS06000
- D7: renamed from D9; Manufacturer (none) -> Würth Elektronik; Part Number (none) -> 151031YS06000
- D8: renamed from D10; Manufacturer (none) -> Würth Elektronik; Part Number (none) -> 151031YS06000
- D9: renamed from D6; value D_Schottky -> BAT43; Manufacturer (none) -> Vishay; Part Number (none) -> BAT43-TAP
- J1: value Conn_01x08_UNO_Digital_1 -> SP-140520-08-001; Manufacturer (none) -> GCT; Part Number (none) -> SP-140520-08-001
- J2: value Conn_01x10_UNO_Digital_2 -> SP-140520-10-001; Manufacturer (none) -> GCT; Part Number (none) -> SP-140520-10-001
- J3: value Conn_01x08_UNO_Power -> SP-140520-08-001; Manufacturer (none) -> GCT; Part Number (none) -> SP-140520-08-001
- J4: value Conn_01x06_UNO_Analog -> SP-140520-06-001; Manufacturer (none) -> GCT; Part Number (none) -> SP-140520-06-001
- J5: value Screw_Terminal_01x03 -> 5430438
- J6: value 6P6C -> 54601-906WPLF
- SW1: renamed from SW2; Manufacturer (none) -> TE; Part Number (none) -> 1825910-6
- SW2: renamed from SW3; Manufacturer (none) -> TE; Part Number (none) -> 1825910-6
- SW3: renamed from SW1; Manufacturer (none) -> TE; Part Number (none) -> 1825910-6
- SW4: value SW_DPDT_x2 -> OS202011MS2QN1
- renumbered R7 to R5, R5 to R6, R8 to R7, R9 to R8, R6 to R9
Connections:
- net +5V: now also C1.1
- net BUTTON1: now also J1.3 (2), SW1.1; no longer J1.4 (3), SW2.1
- net BUTTON2: now also J1.4 (3), SW2.1; no longer J1.3 (2), SW1.1
- net GND: now also C1.2
- net LED1: now also J1.6 (5), R1.1; no longer J2.1 (8), R4.1
- net LED2: now also J1.7 (6), R2.1; no longer J1.8 (7), R3.1
- net LED3: now also J1.8 (7), R3.1; no longer J1.7 (6), R2.1
- net LED4: now also J2.1 (8), R4.1; no longer J1.6 (5), R1.1
Other:
- note added: "All the UNO interface headers can be purchased as Sparkfun PRT-11417."
- moved on the sheet: D1, D2, D3, D4, D5, D7, D8, R1, R2, R3, R4, R5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

Commit message: Updated the main source files.
Parts:
- removed unit 2 of SW4
- C1, C2, C3, C4, C5, C6: symbol Device:C_Polarized_Small -> Project_Symbols:C_Polarized_Small
- D1, D2, D3, D4, D5, D6, D7, D8: symbol Device:LED -> Project_Symbols:LED
- D10, D11, D9: symbol Device:D_Schottky -> Project_Symbols:D_Schottky
- J5: symbol Connector:Screw_Terminal_01x03 -> Project_Symbols:Screw_Terminal_01x03
- J6: symbol Connector:6P6C -> Project_Symbols:6P6C
- R1, R2, R3, R4, R5, R6, R7, R8: symbol Device:R -> Project_Symbols:R; Manufacturer (none) -> Stackpole Electronics; Part Number (none) -> CFM14JT330R
- R9: symbol Device:R -> Project_Symbols:R; Manufacturer (none) -> Stackpole Electronics; Part Number (none) -> CFM14JT10K0
- RV1, RV2: symbol Device:R_Potentiometer -> Project_Symbols:R_Potentiometer
- SW1, SW2, SW3: symbol Switch:SW_Push -> Project_Symbols:SW_Push
- SW4: symbol Switch:SW_DPDT_x2 -> Project_Symbols:SW_DPDT_MountingPin
- U1: value LT1785 -> RS-485 XCVR; symbol Interface_UART:LT1785AxN8 -> Project_Symbols:LT1785AxN8; Manufacturer (none) -> Analog Devices; Part Number (none) -> LT1785ACN8#PBF
- U2: value MAX232 -> RS-232 XCVR; symbol Interface_UART:MAX232 -> Project_Symbols:MAX232; Manufacturer (none) -> Texas Instruments; Part Number (none) -> MAX232N
Connections:
- net GND: now also SW4.MP (MountPin)
- net HARD_TX: now also SW4.4 (A)
- net SOFT_TX: now also SW4.6 (C)
- net TX: now also SW4.5 (B)
Other:
- note added: "Documentation and source files can be found at https://github.com/CMB27/ModbusRTU-Test-Shield."
- company: (none) -> Designer: C. M. Bulliner
- title: (none) -> ModbusRTU Test Shield
- moved on the sheet: C1, C2, C3, C4, C5, C6, D1, D10, D11, D2, D3, D4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
