File: src/ModbusRTU-Test-Shield.kicad_sch (KiCad schematic)
At the start: 40 parts, among them J1 SP-140520-08-001, J2 SP-140520-10-001, J3 SP-140520-08-001, J4 SP-140520-06-001, J5 5430438, J6 54601-906WPLF, SW1 BUTTON1, SW2 BUTTON2, SW3 RESET, SW4 OS202011MS2QN1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

Commit message: Updated the source files.
Other:
- note removed: "All the UNO interface headers can be purchased as Sparkfun PRT-11417."
Changed lines of the file:
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@@
     (effects (font (size 1.27 1.27)) (justify left bottom) (href "https://github.com/CMB27/ModbusRTU-Test-Shield"))
-  )
-  (text "All the UNO interface headers can be purchased as Sparkfun PRT-11417."
-    (at 27.94 88.9 0)
-    (effects (font (size 1.27 1.27)) (justify left bottom))
   )
   (label "HARD_RX" (at 91.44 76.2 0) (fields_autoplaced)
