File: src/ModbusRTU-Test-Shield.kicad_sch (KiCad schematic)
At the start: 40 parts, among them J1 SP-140520-08-001, J2 SP-140520-10-001, J3 SP-140520-08-001, J4 SP-140520-06-001, J5 5430438, J6 54601-906WPLF, SW1 BUTTON1, SW2 BUTTON2, SW3 RESET, SW4 OS202011MS2QN1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

Commit message: Made some changes based on build.
Parts:
- R1, R2, R3, R4, R5, R6, R7, R8: value 330 -> 1K; Part Number CFM14JT330R -> CFM14JT1K00
- SW1, SW2, SW3: Manufacturer TE -> Omron; Part Number 1825910-6 -> B3F-1020
Connections:
- no-connect marks 0 -> 17
Other:
- moved on the sheet: D1, D2, D3, D4, D5, D6, D7, D8, R1, R2, R3, R4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

Commit message: Updated board to 1.0.0. Changed out RJ12 connector for one that is not obsolete. Changed out RS-485 tranceiver for a less expensive model.
Parts:
- J6: value 54601-906WPLF -> RJ12 CONNECTOR; Part Number 54601-906WPLF -> 87180-066LF
- U1: Manufacturer Analog Devices -> Texas Instruments; Part Number LT1785ACN8#PBF -> SN65HVD3082EP
Changed lines of the file:
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@@
   (title_block
     (title "ModbusRTU Test Shield")
-    (date "2024-01-06")
-    (rev "0.1.0")
+    (date "2024-11-29")
+    (rev "1.0.0")
     (company "Designer: C. M. Bulliner")
     (comment 2 "OF MERCHANTABILITY, SATISFACTORY QUALITY AND FITNESS FOR A PARTICULAR PURPOSE.")
@@
       (effects (font (size 1.27 1.27)) hide)
     )
-    (property "Datasheet" "https://www.analog.com/media/en/technical-documentation/data-sheets/LT1785-1785A-1791-1791A.pdf" (at 114.3 170.18 0)
-      (effects (font (size 1.27 1.27)) hide)
-    )
-    (property "Manufacturer" "Analog Devices" (at 101.6 172.72 0)
-      (effects (font (size 1.27 1.27)) hide)
-    )
-    (property "Part Number" "LT1785ACN8#PBF" (at 101.6 172.72 0)
+    (property "Datasheet" "https://www.ti.com/lit/ds/symlink/sn65hvd3082e.pdf?ts=1732870704060&ref_url=https%253A%252F%252Fwww.mouser.es%252F" (at 114.3 170.18 0)
+      (effects (font (size 1.27 1.27)) hide)
+    )
+    (property "Manufacturer" "Texas Instruments" (at 101.6 172.72 0)
+      (effects (font (size 1.27 1.27)) hide)
+    )
+    (property "Part Number" "SN65HVD3082EP" (at 101.6 172.72 0)
       (effects (font (size 1.27 1.27)) hide)
     )
@@
       (effects (font (size 1.27 1.27)) (justify top))
     )
-    (property "Value" "54601-906WPLF" (at 29.21 120.65 90)
+    (property "Value" "RJ12 CONNECTOR" (at 29.21 120.65 90)
       (effects (font (size 1.27 1.27)) (justify bottom))
     )
@@
       (effects (font (size 1.27 1.27)) hide)
     )
-    (property "Datasheet" "https://cdn.amphenol-cs.com/media/wysiwyg/files/drawing/c-bmj-0082.pdf" (at 38.1 120.015 90)
+    (property "Datasheet" "https://cdn.amphenol-cs.com/media/wysiwyg/files/drawing/87180.pdf" (at 38.1 120.015 90)
       (effects (font (size 1.27 1.27)) hide)
     )
@@
       (effects (font (size 1.27 1.27)) hide)
     )
-    (property "Part Number" "54601-906WPLF" (at 38.1 119.38 0)
-      (effects (font (size 1.27 1.27)) hide)
-    )
+    (property "Part Number" "87180-066LF" (at 38.1 119.38 0)
+      (effects (font (size 1.27 1.27)) hide)
+    )
